File: kicad proyecto.kicad_sch (KiCad schematic)
At the start: 45 parts, among them J1 USB_B, J2 UART, Q1 MMBT3904, SW1 SW_SPST, SW2 SW_SPST, SW3 SW_SPST, U1 NE555D, U2 NE555D, U3 FT232RL, U4 LM741, U5 4040, U6 4040

Commit message: Add files via upload
Connections:
- net USB_D-: now reaches J1.2 (D-), U3.16 (USBD-)
- net USB_D+: now reaches J1.3 (D+), U3.15 (USBD+)
Changed lines of the file:
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@@
+	(wire
+		(pts
+			(xy 146.05 127) (xy 154.94 127)
+		)
+		(stroke
+			(width 0)
+			(type default)
+		)
+	)
 	(wire
 		(pts
@@
 	(wire
 		(pts
-			(xy 146.05 127) (xy 154.94 127)
-		)
-		(stroke
-			(width 0)
-			(type default)
-		)
-	)
-	(wire
-		(pts
 			(xy 175.26 67.31) (xy 175.26 71.12)
 		)
@@
 	(wire
 		(pts
+			(xy 146.05 124.46) (xy 154.94 124.46)
+		)
+		(stroke
+			(width 0)
+			(type default)
+		)
+	)
+	(wire
+		(pts
 			(xy 26.67 43.18) (xy 26.67 44.45)
 		)
@@
 	(wire
 		(pts
-			(xy 146.05 124.46) (xy 154.94 124.46)
-		)
-		(stroke
-			(width 0)
-			(type default)
-		)
-	)
-	(wire
-		(pts
 			(xy 44.45 45.72) (xy 44.45 78.74)
 		)
@@
 		)
 	)
+	(label "USB_D+"
+		(at 148.59 124.46 0)
+		(effects
+			(font
+				(size 1.27 1.27)
+			)
+			(justify left bottom)
+		)
+	)
+	(label "USB_D-"
+		(at 152.4 127 0)
+		(effects
+			(font
+				(size 1.27 1.27)
+			)
+			(justify left bottom)
+		)
+	)

Commit message: Add files via upload
Connections:
- net USB_D+ renamed USB_D P
- net USB_D- renamed USB_D N
Changed lines of the file:
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@@
 		)
 	)
-	(label "USB_D+"
-		(at 148.59 124.46 0)
+	(label "USB_D P"
+		(at 147.32 124.46 0)
 		(effects
 			(font
@@
 		)
 	)
-	(label "USB_D-"
-		(at 152.4 127 0)
+	(label "USB_D N"
+		(at 147.32 127 0)
 		(effects
 			(font

Commit message: Add files via upload
Parts:
- 10k1, 50k1: footprint Potentiometer_THT:Potentiometer_ACP_CA6-H2,5_Horizontal -> pretty:601030
Changed lines of the file:
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@@
 			)
 		)
-		(property "Footprint" "Potentiometer_THT:Potentiometer_ACP_CA6-H2,5_Horizontal"
+		(property "Footprint" "pretty:601030"
 			(at 76.2 146.05 0)
 			(effects
@@
 			)
 		)
-		(property "Footprint" "Potentiometer_THT:Potentiometer_ACP_CA6-H2,5_Horizontal"
+		(property "Footprint" "pretty:601030"
 			(at 101.6 59.69 0)
 			(effects
